File: hardware/telescopeheater.kicad_pcb (KiCad board)
At the start: 2 copper layers, 77.5 x 20.3 mm, 19 parts, among them IC1 ATTINY25-S, P1 Power, P2 ISP, P3 Heater, P4 Heater, Q1 IRLML0030, Q2 IRLML0030, U1 LP2985LV

Commit message: fix MOSFET footprint
Parts:
- Q1, Q2: footprint TO_SOT_Packages_SMD:SOT-23 -> heater:SOT-23-IRLM
- moved R2 3.70 mm to (113.7, 108.6), turned to 0 degrees
- moved R1 3.18 mm to (141.0, 104.8)
- moved Q1 2.54 mm to (138.4, 102.9), turned to 180 degrees
- moved Q2 1.42 mm to (111.8, 106.0), turned to 180 degrees
Routing:
- net GND: track 171.6 -> 192.4 mm, vias 2 -> 1
- net Net-(D1-Pad1): track 7.31 -> 17.0 mm
- net Net-(IC1-Pad5): track 41.7 -> 44.5 mm
- net Net-(D2-Pad1): track 9.37 -> 7.44 mm
- net Net-(IC1-Pad6): track 27.2 -> 26.3 mm
- net Net-(Q2-Pad3): track 2.38 -> 1.67 mm
