File: hardware/telescopeheater.sch (KiCad schematic (older format))
At the start: 20 parts, among them IC1 ATTINY25-S, P1 Power, P2 ISP, P3 Heater, P4 Heater, Q1 IRLML0030, Q2 IRLML0030, U1 LP2985LV

Commit message: first version
Parts:
- removed C2: 1u, symbol CP
- C1: footprint (none) -> Capacitors_Tantalum_SMD:CP_Tantalum_Case-C_EIA-6032-28_Hand
- C2: renamed from C4; value 3.3n -> 4.7u; footprint (none) -> Capacitors_SMD:C_0805_HandSoldering
- C3: footprint (none) -> Capacitors_SMD:C_0603_HandSoldering
- D1, D2: footprint (none) -> LEDs:LED_D3.0mm
- IC1: footprint SO8-200 -> Housings_SOIC:SSO-8_6.8x5.9mm_Pitch1.27mm_Clearance7mm
- P1: footprint (none) -> heater:Power
- P2: footprint (none) -> heater:ISP
- P3, P4: footprint (none) -> heater:RC-5231
- Q1, Q2: footprint (none) -> TO_SOT_Packages_SMD:SOT-23
- R1, R2, R3, R4: footprint (none) -> Resistors_SMD:R_0603_HandSoldering
- RV1, RV2: footprint (none) -> heater:Cermet
- U1: footprint (none) -> TO_SOT_Packages_SMD:SOT-23-5_HandSoldering
Changed lines of the file:
@@
 LIBS:contrib
 LIBS:valves
+LIBS:telescopeheater-cache
 EELAYER 25 0
 EELAYER END
@@
 F 0 "IC1" H 4900 4150 50  0000 C CNN
 F 1 "ATTINY25-S" H 7050 3350 50  0000 C CNN
-F 2 "SO8-200" H 7000 3750 50  0000 C CIN
+F 2 "Housings_SOIC:SSO-8_6.8x5.9mm_Pitch1.27mm_Clearance7mm" H 7000 3750 50  0000 C CIN
 F 3 "" H 6050 3750 50  0000 C CNN
 	1    6050 3750
@@
 F 0 "C3" H 7725 3750 50  0000 L CNN
 F 1 "0.1u" H 7725 3550 50  0000 L CNN
-F 2 "" H 7738 3500 50  0000 C CNN
+F 2 "Capacitors_SMD:C_0603_HandSoldering" H 7738 3500 50  0001 C CNN
 F 3 "" H 7700 3650 50  0000 C CNN
 	1    7700 3650
@@
 F 0 "RV2" V 725 4050 50  0000 C CNN
 F 1 "100k" V 800 4050 50  0000 C CNN
-F 2 "" H 900 4050 50  0000 C CNN
+F 2 "heater:Cermet" H 900 4050 50  0001 C CNN
 F 3 "" H 900 4050 50  0000 C CNN
 	1    900  4050
@@
 F 0 "R4" V 1280 4050 50  0000 C CNN
 F 1 "10k" V 1200 4050 50  0000 C CNN
-F 2 "" V 1130 4050 50  0000 C CNN
+F 2 "Resistors_SMD:R_0603_HandSoldering" V 1130 4050 50  0001 C CNN
 F 3 "" H 1200 4050 50  0000 C CNN
 	1    1200 4050
@@
 F 0 "P2" H 2750 6500 50  0000 C CNN
 F 1 "ISP" H 2750 6100 50  0000 C CNN
-F 2 "" H 2750 5100 50  0000 C CNN
+F 2 "heater:ISP" H 2750 5100 50  0001 C CNN
 F 3 "" H 2750 5100 50  0000 C CNN
 	1    2750 6300
@@
 F 0 "P1" H 10000 1500 50  0000 C CNN
 F 1 "Power" V 10100 1350 50  0000 C CNN
-F 2 "" H 10000 1350 50  0000 C CNN
+F 2 "heater:Power" H 10000 1350 50  0001 C CNN
 F 3 "" H 10000 1350 50  0000 C CNN
 	1    10000 1350
@@
 F 0 "C1" H 9325 1550 50  0000 L CNN
 F 1 "10u" H 9325 1350 50  0000 L CNN
-F 2 "" H 9338 1300 50  0000 C CNN
+F 2 "Capacitors_Tantalum_SMD:CP_Tantalum_Case-C_EIA-6032-28_Hand" H 9338 1300 50  0001 C CNN
 F 3 "" H 9300 1450 50  0000 C CNN
 	1    9300 1450
@@
 F 0 "Q2" H 2650 1900 50  0000 L CNN
 F 1 "IRLML0030" H 2650 1800 50  0000 L CNN
-F 2 "" H 2650 1950 50  0000 C CNN
+F 2 "TO_SOT_Packages_SMD:SOT-23" H 2650 1950 50  0001 C CNN
 F 3 "" H 2450 1850 50  0000 C CNN
 	1    2450 1850
@@
 F 0 "D2" H 2550 1600 50  0000 C CNN
 F 1 "HLMP-1601" H 2550 1400 50  0000 C CNN
-F 2 "" H 2550 1500 50  0000 C CNN
+F 2 "LEDs:LED_D3.0mm" H 2550 1500 50  0001 C CNN
 F 3 "" H 2550 1500 50  0000 C CNN
 	1    2550 1500
@@
 F 0 "P4" H 3250 1750 50  0000 C CNN
 F 1 "Heater" V 3350 1600 50  0000 C CNN
-F 2 "" H 3250 1600 50  0000 C CNN
+F 2 "heater:RC-5231" H 3250 1600 50  0001 C CNN
 F 3 "" H 3250 1600 50  0000 C CNN
 	1    3250 1600
@@
 F 0 "R2" V 2180 1850 50  0000 C CNN
 F 1 "1k" V 2100 1850 50  0000 C CNN
-F 2 "" V 2030 1850 50  0000 C CNN
+F 2 "Resistors_SMD:R_0603_HandSoldering" V 2030 1850 50  0001 C CNN
 F 3 "" H 2100 1850 50  0000 C CNN
 	1    2100 1850
@@
 F 0 "Q1" H 4350 1900 50  0000 L CNN
 F 1 "IRLML0030" H 4350 1800 50  0000 L CNN
-F 2 "" H 4350 1950 50  0000 C CNN
+F 2 "TO_SOT_Packages_SMD:SOT-23" H 4350 1950 50  0001 C CNN
 F 3 "" H 4150 1850 50  0000 C CNN
 	1    4150 1850
@@
 F 0 "D1" H 4250 1600 50  0000 C CNN
 F 1 "HLMP-1601" H 4250 1400 50  0000 C CNN
-F 2 "" H 4250 1500 50  0000 C CNN
+F 2 "LEDs:LED_D3.0mm" H 4250 1500 50  0001 C CNN
 F 3 "" H 4250 1500 50  0000 C CNN
 	1    4250 1500
@@
 F 0 "P3" H 4950 1750 50  0000 C CNN
 F 1 "Heater" V 5050 1600 50  0000 C CNN
-F 2 "" H 4950 1600 50  0000 C CNN
+F 2 "heater:RC-5231" H 4950 1600 50  0001 C CNN
 F 3 "" H 4950 1600 50  0000 C CNN
 	1    4950 1600
@@
 F 0 "R1" V 3880 1850 50  0000 C CNN
 F 1 "1k" V 3800 1850 50  0000 C CNN
-F 2 "" V 3730 1850 50  0000 C CNN
+F 2 "Resistors_SMD:R_0603_HandSoldering" V 3730 1850 50  0001 C CNN
 F 3 "" H 3800 1850 50  0000 C CNN
 	1    3800 1850
@@
 F 0 "RV1" V 725 3300 50  0000 C CNN
 F 1 "100k" V 800 3300 50  0000 C CNN
-F 2 "" H 900 3300 50  0000 C CNN
+F 2 "heater:Cermet" H 900 3300 50  0001 C CNN
 F 3 "" H 900 3300 50  0000 C CNN
 	1    900  3300
@@
 F 0 "R3" V 1280 3300 50  0000 C CNN
 F 1 "10k" V 1200 3300 50  0000 C CNN
-F 2 "" V 1130 3300 50  0000 C CNN
+F 2 "Resistors_SMD:R_0603_HandSoldering" V 1130 3300 50  0001 C CNN
 F 3 "" H 1200 3300 50  0000 C CNN
 	1    1200 3300
@@
 F 0 "U1" H 8100 1150 50  0000 C CNN
 F 1 "LP2985LV" H 7900 2050 50  0000 C CNN
-F 2 "" H 7900 1600 50  0000 C CNN
+F 2 "TO_SOT_Packages_SMD:SOT-23-5_HandSoldering" H 7900 1600 50  0001 C CNN
 F 3 "" H 7900 1600 50  0000 C CNN
 	1    7900 1600
@@
 $EndComp
 $Comp
-L CP C2
-U 1 1 5A60DAB6
-P 6600 1450
-F 0 "C2" H 6625 1550 50  0000 L CNN
-F 1 "1u" H 6625 1350 50  0000 L CNN
-F 2 "" H 6638 1300 50  0000 C CNN
-F 3 "" H 6600 1450 50  0000 C CNN
-	1    6600 1450
-	1    0    0    -1
-$EndComp
-$Comp
-L C C4
+L C C2
 U 1 1 5A60DB33
 P 6900 1450
-F 0 "C4" H 6925 1550 50  0000 L CNN
-F 1 "3.3n" H 6925 1350 50  0000 L CNN
-F 2 "" H 6938 1300 50  0000 C CNN
+F 0 "C2" H 6925 1550 50  0000 L CNN
+F 1 "4.7u" H 6925 1350 50  0000 L CNN
+F 2 "Capacitors_SMD:C_0805_HandSoldering" H 6938 1300 50  0001 C CNN
 F 3 "" H 6900 1450 50  0000 C CNN
 	1    6900 1450
@@
 	1    0    0    -1
 $EndComp
-$Comp
-L GND #PWR021
-U 1 1 5A60DC62
-P 6600 1600
-F 0 "#PWR021" H 6600 1350 50  0001 C CNN
-F 1 "GND" H 6600 1450 50  0000 C CNN
-F 2 "" H 6600 1600 50  0000 C CNN
-F 3 "" H 6600 1600 50  0000 C CNN
-	1    6600 1600
-	1    0    0    -1
-$EndComp
-Wire Wire Line
-	6600 1300 7100 1300
 Connection ~ 6900 1300
 $Comp
-L +5V #PWR022
+L +5V #PWR021
 U 1 1 5A60DD18
-P 6600 1300
-F 0 "#PWR022" H 6600 1150 50  0001 C CNN
-F 1 "+5V" H 6600 1440 50  0000 C CNN
-F 2 "" H 6600 1300 50  0000 C CNN
-F 3 "" H 6600 1300 50  0000 C CNN
-	1    6600 1300
-	1    0    0    -1
-$EndComp
+P 6900 1300
+F 0 "#PWR021" H 6900 1150 50  0001 C CNN
+F 1 "+5V" H 6900 1440 50  0000 C CNN
+F 2 "" H 6900 1300 50  0000 C CNN
+F 3 "" H 6900 1300 50  0000 C CNN
+	1    6900 1300
+	1    0    0    -1
+$EndComp
+Wire Wire Line
+	7100 1300 6900 1300
 $EndSCHEMATC

Commit message: fix MOSFET footprint
Parts:
- Q1, Q2: footprint TO_SOT_Packages_SMD:SOT-23 -> heater:SOT-23-IRLM
Changed lines of the file:
@@
 F 0 "Q2" H 2650 1900 50  0000 L CNN
 F 1 "IRLML0030" H 2650 1800 50  0000 L CNN
-F 2 "TO_SOT_Packages_SMD:SOT-23" H 2650 1950 50  0001 C CNN
+F 2 "heater:SOT-23-IRLM" H 2650 1950 50  0001 C CNN
 F 3 "" H 2450 1850 50  0000 C CNN
 	1    2450 1850
@@
 F 0 "Q1" H 4350 1900 50  0000 L CNN
 F 1 "IRLML0030" H 4350 1800 50  0000 L CNN
-F 2 "TO_SOT_Packages_SMD:SOT-23" H 4350 1950 50  0001 C CNN
+F 2 "heater:SOT-23-IRLM" H 4350 1950 50  0001 C CNN
 F 3 "" H 4150 1850 50  0000 C CNN
 	1    4150 1850
